Commit message: align Go2-X5 assets and cameras with PCT

File: conveyor_bench/assets/robots/go2_x5/go2_x5.urdf (robot description, URDF)
Before this commit: robot go2_x5, 53 links, 52 joints
Links:
- link Head_lower: geometry collision sphere radius=0.047
- link Head_upper: geometry collision cylinder length=0.09 radius=0.05
- link arm_base_link: mass 0.428 -> 0.43995; geometry collision mesh filename=./meshes/X5/base_link.STL; visual mesh filename=./meshes/X5/base_link.STL
- link arm_link1: mass 0.064 -> 0.066982; geometry collision mesh filename=./meshes/X5/link1.STL; visual mesh filename=./meshes/X5/link1.STL
- link arm_link2: mass 1.165 -> 1.0795; geometry collision mesh filename=./meshes/X5/link2.STL; visual mesh filename=./meshes/X5/link2.STL
- link arm_link3: mass 0.546 -> 0.54534; geometry collision mesh filename=./meshes/X5/link3.STL; visual mesh filename=./meshes/X5/link3.STL
- link arm_link4: mass 0.100 -> 0.11714; geometry collision mesh filename=./meshes/X5/link4.STL; visual mesh filename=./meshes/X5/link4.STL
- link arm_link5: mass 0.655 -> 0.63488; geometry collision mesh filename=./meshes/X5/link5.STL; visual mesh filename=./meshes/X5/link5.STL
- link arm_link6: mass 0.902 -> 0.44089; geometry collision mesh filename=./meshes/X5/link6.STL; visual mesh filename=./meshes/X5/link6.STL
Joints:
- joint arm_base_joint: origin xyz=0.085 0 0.094 rpy=0 0 0 -> xyz=0.12 0 0.05 rpy=0 0 0
- joint arm_joint1: limit lower=-3.14159265359 upper=3.14159265359 effort=30 velocity=10 -> lower=-2.618 upper=3.14 effort=15 velocity=3; origin xyz=0 0 0.0603 rpy=0 0 0 -> xyz=0 0 0.0605 rpy=0 0 0
- joint arm_joint2: limit lower=0 upper=3.66519 effort=30 velocity=10 -> lower=0 upper=3.14 effort=15 velocity=3; origin xyz=0.02 0 0.0402 rpy=0 0 0 -> xyz=0.02 0 0.04 rpy=0 0 0
- joint arm_joint3: limit lower=0 upper=3.14159265359 effort=30 velocity=10 -> lower=0 upper=3.14 effort=15 velocity=3; origin xyz=-0.264 0 0 rpy=-3.1416 0 0 -> xyz=-0.264 0 0 rpy=3.1416 0 0
- joint arm_joint4: limit lower=-1.57079632679 upper=1.57079632679 effort=30 velocity=10 -> lower=-1.5708 upper=1.5708 effort=3 velocity=3
- joint arm_joint5: limit lower=-1.57079632679 upper=1.57079632679 effort=30 velocity=10 -> lower=-1.5708 upper=1.5708 effort=3 velocity=3; origin xyz=0.06575 -0.001 -0.0825 rpy=0 0 0 -> xyz=0.06775 0.0005 -0.0865 rpy=0 0 0
- joint arm_joint6: limit lower=-1.57079632679 upper=1.57079632679 effort=30 velocity=10 -> lower=-1.5708 upper=1.5708 effort=3 velocity=3; origin xyz=0.02845 0 0.0825 rpy=-3.1416 0 0 -> xyz=0.02895 0 0.0865 rpy=-3.1416 0 0
- joint grasp_tcp_fixed_joint: origin xyz=0.125 0.0 0.0 rpy=0 0 0 -> xyz=0.15757 0.0 0.0 rpy=0 0 0
